File: Hardware/ElectroLab.brd (EAGLE design)
At the start: 175 x 100 mm, 230 parts, among them IC1 LM2902DT, IC10 CD4511BNSR, IC11 PAM8403, IC13 ADXL337, IC14 MIC5205, IC2 LM2902DT, IC3 SN74LV08ADR, IC4 SN74LV32ADR, IC5 SN74LV04ADR, IC6 4027D, IC7 4027D, IC8 NE555D, IC9 AT42QT1012, U1 USB, U2 USB-B

Commit message: Update modifications for ElectroLab R2 CTI20 Release
Parts:
- moved C1 0.68 mm to (33.4, 37.8)
- moved C11 0.68 mm to (33.4, 25.1)
- moved C13 0.68 mm to (33.4, 22.5)
- moved C15 0.68 mm to (33.4, 20.0)
- moved C17 0.68 mm to (33.4, 17.5)
- moved C3 0.68 mm to (33.4, 35.2)
- moved C35 0.68 mm to (33.6, 8.50)
- moved C5 0.68 mm to (33.4, 32.7)
- moved C7 0.68 mm to (33.4, 30.1)
- moved C9 0.68 mm to (33.4, 27.6)
- moved PH50 0.68 mm to (19.5, 52.3)
- moved PH51 0.68 mm to (29.5, 52.3)
- moved PH52 0.68 mm to (32.2, 52.3)
- moved PH53 0.68 mm to (42.2, 52.3)
- moved PH57 0.68 mm to (40.2, 26.3)
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Routing:
- net VCC: track 466.5 -> 457.7 mm, vias 13 -> 12
- net N$70: track 9.67 -> 4.46 mm
- net N$80: track 9.14 -> 3.93 mm
- net N$117: track 8.17 -> 5.58 mm
- net GND: track 66.7 -> 64.3 mm, vias 19 -> 16
- net SENSE: track 7.72 -> 9.82 mm, vias 2 -> 1
- net D12: track 33.0 -> 32.2 mm
Other:
- board text added: "0000-0 0001-1 0010-2 0011-3 0100-4 0101-5 0110-6 0111-7 1000-8 1001-9"
- board text added: "100"
- board text added: "100K"
- board text added: "100n"
- board text added: "100p"
- board text added: "100u"
- board text added: "10K"
- board text added: "10n"
- board text added: "10p"
- board text added: "10u"
- board text added: "15K"
- board text added: "1K"
- board text added: "1m"
- board text added: "1n"
- board text added: "1u"
- board text added: "4.7K"
- board text added: "470"
- board text added: "470K"
- board text added: "47K"
- board text added: "50n"
- board text added: "AUX"
- board text added: "ArduLab"
- board text added: "Blue"
- board text added: "DIS"
- board text added: "Dig 1"
- board text added: "Dig 2"
- board text added: "Green"
- board text added: "J"
- board text added: "K"
- board text added: "L"
- board text added: "NPN"
- board text added: "NTC"
- board text added: "OUT"
- board text added: "PNP"
- board text added: "Power"
- board text added: "Q"
- board text added: "R"
- board text added: "Red"
- board text added: "THR"
- board text added: "TRIG"
- board text added: "USB"
- board text added: "X"
- board text added: "Y"
- board text added: "Z"

Commit message: Updated BRD with manufactured silkscreen R2
Parts:
- moved C1 0.68 mm to (34.1, 37.8)
- moved C11 0.68 mm to (34.1, 25.1)
- moved C13 0.68 mm to (34.1, 22.5)
- moved C15 0.68 mm to (34.1, 20.0)
- moved C17 0.68 mm to (34.1, 17.5)
- moved C3 0.68 mm to (34.1, 35.2)
- moved C35 0.68 mm to (34.3, 8.50)
- moved C5 0.68 mm to (34.1, 32.7)
- moved C7 0.68 mm to (34.1, 30.1)
- moved C9 0.68 mm to (34.1, 27.6)
- moved PH50 0.68 mm to (20.1, 52.3)
- moved PH51 0.68 mm to (30.1, 52.3)
- moved PH52 0.68 mm to (32.9, 52.3)
- moved PH53 0.68 mm to (42.9, 52.3)
- moved PH57 0.68 mm to (40.9, 26.3)
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Routing:
- net VCC: track 457.7 -> 466.5 mm, vias 12 -> 13
- net N$70: track 4.46 -> 9.67 mm
- net N$80: track 3.93 -> 9.14 mm
- net N$117: track 5.58 -> 8.17 mm
- net GND: track 64.3 -> 66.7 mm, vias 16 -> 19
- net SENSE: track 9.82 -> 7.72 mm, vias 1 -> 2
- net D12: track 32.2 -> 33.0 mm
Other:
- board text removed: "0000-0 0001-1 0010-2 0011-3 0100-4 0101-5 0110-6 0111-7 1000-8 1001-9"
- board text removed: "100"
- board text removed: "100K"
- board text removed: "100n"
- board text removed: "100p"
- board text removed: "100u"
- board text removed: "10K"
- board text removed: "10n"
- board text removed: "10p"
- board text removed: "10u"
- board text removed: "15K"
- board text removed: "1K"
- board text removed: "1m"
- board text removed: "1n"
- board text removed: "1u"
- board text removed: "4.7K"
- board text removed: "470"
- board text removed: "470K"
- board text removed: "47K"
- board text removed: "50n"
- board text removed: "AUX"
- board text removed: "ArduLab"
- board text removed: "Blue"
- board text removed: "DIS"
- board text removed: "Dig 1"
- board text removed: "Dig 2"
- board text removed: "Green"
- board text removed: "J"
- board text removed: "K"
- board text removed: "L"
- board text removed: "NPN"
- board text removed: "NTC"
- board text removed: "OUT"
- board text removed: "PNP"
- board text removed: "Power"
- board text removed: "Q"
- board text removed: "R"
- board text removed: "Red"
- board text removed: "THR"
- board text removed: "TRIG"
- board text removed: "USB"
- board text removed: "X"
- board text removed: "Y"
- board text removed: "Z"

Commit message: First R3 version before merging silkscreen layers
Parts:
- removed C28: 10nF, SpaceDIY_passive_components:0603
- removed IC9: AT42QT1012, SparkFun-Sensors:SOT-23-6
- removed PH13: (no value), pinhead:1X03
- removed RGB: (no value), Passive_components:PLCC6
- removed U$15: CAPACITIVE_SENSOR_PAD, SpaceDIY:CAPACITIVE_SENSOR_PAD
- added F1: 500mA, adafruit:R1206
- added JC2: SWTCHCRFT_3.5JACK5-JACK-SMD, jmsaavedra:4-JACK-SMD
- added L17: Grn, adafruit:1206
- added LED_: (no value), SpaceDIY_passive_components:PLCC-6
- added PH34: (no value), pinhead:1X01
- added PH64: (no value), pinhead:1X03
- added PH65: (no value), pinhead:1X04
- C21, C23, C24, C25, C26: device resistor:C1206 -> SpaceDIY_passive_components:0603
- C22: value 100n -> 470n
- JC1: value (none) -> SWTCHCRFT_3.5JACK5-JACK-SMD
- NTC: device adafruit:R1206 -> adafruit:R1206@1
- PH21: device pinhead:1X03 -> pinhead:1X02
- PH31: device pinhead:1X04 -> pinhead:1X30
- PH38: device pinhead:1X06 -> pinhead:1X03
- R39: value 100k -> 330; device SpaceDIY_passive_components:0603 -> resistor:R1206
- R40: value 1M -> 10k
- R60: device resistor:R1206 -> SpaceDIY_passive_components:0603
- U2: value USB-B -> GAS_SENSOR; device SparkFun-Connectors:USB-B-PTH -> SparkFun:MQ-3
- moved C27 132.9 mm to (143.3, 3.70)
- moved C25 125.3 mm to (148.6, 8.56), turned to 90 degrees
- moved C23 123.3 mm to (138.2, 11.7)
- moved R60 123.3 mm to (149.6, 4.94)
- moved IC11 122.5 mm to (143.4, 12.0)
- moved C26 122.4 mm to (151.3, 4.94)
- moved C24 121.3 mm to (148.5, 11.6), turned to 90 degrees
- moved PH38 94.1 mm to (136.1, 12.0), turned to 90 degrees
- moved U2 94.1 mm to (87.5, 30.4), turned to 0 degrees
- moved R39 86.5 mm to (171.1, 11.3), turned to 0 degrees
- moved R40 68.2 mm to (137.4, 4.90)
- moved C22 63.7 mm to (135.6, 4.90), turned to 270 degrees
- moved PH31 23.6 mm to (89.3, 67.2), turned to 0 degrees
- moved PH35 23.3 mm to (119.0, 81.2)
- moved PH21 20.2 mm to (87.5, 18.8)
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Connections:
- removed net +OUT: IC11.16, PH38.5
- removed net -OUT: IC11.14, PH38.6
- removed net IN: C26.1, PH38.1
- removed net N$258: PH59.1, PH60.1, PH61.1
- removed net N$259: PH59.2, PH60.2, PH61.2
- removed net N$260: PH59.3, PH60.3, PH61.3
- removed net N$261: PH59.4, PH60.4, PH61.4
- removed net N$265: PH59.5, PH60.5, PH61.5
- removed net N$266: PH59.6, PH60.6, PH61.6
- removed net N$267: PH59.7, PH60.7, PH61.7
- removed net N$268: PH59.8, PH60.8, PH61.8
- removed net N$269: PH59.9, PH60.9, PH61.9
- removed net N$270: PH59.10, PH60.10, PH61.10
- removed net N$271: PH59.11, PH60.11, PH61.11
- removed net N$272: PH59.12, PH60.12, PH61.12
- removed net N$273: PH59.13, PH60.13, PH61.13
- removed net N$274: PH59.14, PH60.14, PH61.14
- removed net N$275: PH59.15, PH60.15, PH61.15
- removed net N$276: PH59.16, PH60.16, PH61.16
- removed net N$277: PH59.17, PH60.17, PH61.17
- removed net N$278: PH59.18, PH60.18, PH61.18
- removed net N$279: PH59.19, PH60.19, PH61.19
- removed net N$280: PH59.20, PH60.20, PH61.20
- removed net N$281: PH59.21, PH60.21, PH61.21
- removed net N$282: PH59.22, PH60.22, PH61.22
- removed net N$283: PH59.23, PH60.23, PH61.23
- removed net N$284: PH59.24, PH60.24, PH61.24
- removed net N$285: PH59.25, PH60.25, PH61.25
- removed net N$286: PH59.26, PH60.26, PH61.26
- removed net N$287: PH59.27, PH60.27, PH61.27
- removed net N$288: PH59.28, PH60.28, PH61.28
- removed net N$289: PH59.29, PH60.29, PH61.29
- removed net N$290: PH59.30, PH60.30, PH61.30
- removed net OUT01: IC9.1, PH21.2, R39.2
- removed net PVDD: C23.1, C24.1, C27.+, IC11.13, IC11.4, IC11.6, PH38.3
- removed net SENSE: R67.1, U$15.0
- removed net SNS: C28.2, IC9.4, R40.2
- removed net SNSK: C28.1, IC9.3, R67.2
- new net INL: IC11.7, R60.1
- new net IN_L: C26.1, PH38.3
- new net IN_R: C22.1, PH38.2
- new net JC2: JC2.2, PH64.2
- new net N$118: F1.1, S1.2
- new net N$119: PH34.1, R67.2, U2.B1
- new net N$120: JC2.1, PH64.3
- new net N$121: JC2.3, PH64.1
- new net N$122: L17.A, R39.1
- new net N$124: C22.2, R40.2
- new net N$127: PH31.7, PH59.7, PH60.7, PH61.7
- new net N$128: PH31.1, PH59.1, PH60.1, PH61.1
- new net N$129: PH31.2, PH59.2, PH60.2, PH61.2
- new net N$139: PH31.3, PH59.3, PH60.3, PH61.3
- new net N$140: PH31.4, PH59.4, PH60.4, PH61.4
- new net N$141: PH31.5, PH59.5, PH60.5, PH61.5
- new net N$142: PH31.6, PH59.6, PH60.6, PH61.6
- new net N$143: PH31.8, PH59.8, PH60.8, PH61.8
- new net N$144: PH31.9, PH59.9, PH60.9, PH61.9
- new net N$145: PH31.10, PH59.10, PH60.10, PH61.10
- new net N$147: PH31.11, PH59.11, PH60.11, PH61.11
- new net N$148: PH31.12, PH59.12, PH60.12, PH61.12
- new net N$149: PH31.13, PH59.13, PH60.13, PH61.13
- new net N$150: PH31.14, PH59.14, PH60.14, PH61.14
- new net N$151: PH31.15, PH59.15, PH60.15, PH61.15
- new net N$152: PH31.16, PH59.16, PH60.16, PH61.16
- new net N$153: PH31.17, PH59.17, PH60.17, PH61.17
- new net N$154: PH31.18, PH59.18, PH60.18, PH61.18
- new net N$163: PH31.19, PH59.19, PH60.19, PH61.19
- new net N$164: PH31.20, PH59.20, PH60.20, PH61.20
- new net N$165: PH31.21, PH59.21, PH60.21, PH61.21
- new net N$166: PH31.22, PH59.22, PH60.22, PH61.22
- new net N$167: PH31.23, PH59.23, PH60.23, PH61.23
- new net N$168: PH31.24, PH59.24, PH60.24, PH61.24
- new net N$169: PH31.25, PH59.25, PH60.25, PH61.25
- new net N$170: PH31.26, PH59.26, PH60.26, PH61.26
- new net N$174: PH31.27, PH59.27, PH60.27, PH61.27
- new net N$175: PH31.28, PH59.28, PH60.28, PH61.28
- new net N$176: PH31.29, PH59.29, PH60.29, PH61.29
- new net N$177: PH31.30, PH59.30, PH60.30, PH61.30
- new net OUT_L+: IC11.1, PH65.4
- new net OUT_L-: IC11.3, PH65.3
- new net OUT_R+: IC11.16, PH65.2
- new net OUT_R-: IC11.14, PH65.1
- net GND: now also L17.C, LED_.4, LED_.5, LED_.6, PH38.1, R67.1, U2.HB; no longer C22.2, IC9.2, IC9.6, PH38.2, PH38.4, R39.1, R40.1, RGB.B-, RGB.G-, RGB.R-, U2.GND
- net INR: now also R40.1; no longer R60.1
- net N$117: now also LED_.2; no longer RGB.G+
- net N$126: now also PH21.2; no longer PH21.3
- net N$224: now also R39.2
- net N$308: now also LED_.1; no longer RGB.R+
- net N$310: now also LED_.3; no longer RGB.B+
- net SA': no longer PH31.1
- net SB': no longer PH13.1
- net SC': no longer PH13.3
- net SD': no longer PH31.4
- net SE': no longer PH31.3
- net SF': no longer PH31.2
- net SG': no longer PH13.2
- net VCC: now also C23.1, C24.1, C27.+, F1.2, IC11.13, IC11.4, IC11.6, U2.A1, U2.HA; no longer C22.1, IC9.5, S1.2
- net VUSB: no longer U2.VBUS
Routing:
- net PVDD: track 52.6 -> 0.00 mm, vias 2 -> 0
- net -OUT: track 46.6 -> 0.00 mm, vias 2 -> 0
- net +OUT: track 36.4 -> 0.00 mm
- net SF': track 62.1 -> 26.4 mm
- net SG': track 53.5 -> 18.3 mm, vias 4 -> 2
- net GND: track 66.7 -> 33.1 mm, vias 19 -> 14
- net IA: track 11.7 -> 43.4 mm, vias 0 -> 2
- net SB': track 40.6 -> 9.96 mm, vias 2 -> 0
- net SE': track 50.0 -> 19.5 mm, vias 3 -> 2
- net N$125: track 32.7 -> 2.22 mm
- net N$126: track 32.7 -> 2.26 mm
- net N$120: track 0.00 -> 26.8 mm
- net SC': track 41.9 -> 15.7 mm
- net VCC: track 466.5 -> 491.8 mm, vias 13 -> 14
- net VUSB: track 37.3 -> 13.6 mm
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Other:
- board text removed: "5V"
- board text removed: "ACC"
- board text removed: "D10"
- board text removed: "D11"
- board text removed: "D12"
- board text removed: "D13"
- board text removed: "D9"
- board text removed: "GND"
- board text removed: "IN"
- board text removed: "OUT+"
- board text removed: "OUT-"
- board text removed: "U2"

Commit message: Updated to R3 (Mk.III)
Connections:
- net G: now also R57.2; no longer R58.2
- net R: now also R58.2; no longer R57.2
Routing:
- net G: track 14.9 -> 4.89 mm, vias 1 -> 0
- net R: track 4.76 -> 9.81 mm
- net N$103: track 4.97 -> 3.28 mm
