File: Hardware/ElectroLab.sch (EAGLE design)
At the start: 230 parts, among them IC1 LM2902DT, IC10 CD4511BNSR, IC11 PAM8403, IC13 ADXL337, IC14 MIC5205, IC2 LM2902DT, IC3 SN74LV08ADR, IC4 SN74LV32ADR, IC5 SN74LV04ADR, IC6 4027D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

Commit message: First R3 version before merging silkscreen layers
Parts:
- removed C28: 10nF, SpaceDIY_passive_components:C0603
- removed IC9: AT42QT1012, SparkFun-Sensors:AT42QT1012
- removed PH13: (no value), pinhead:PINHD-1X3
- removed RGB: LED_RGB_PLCC6, Passive_components:LED_RGB_PLCC6
- removed U$15: CAPACITIVE_SENSOR_PAD, SpaceDIY:CAPACITIVE_SENSOR_PAD
- added F1: 500mA, adafruit:PTCFUSE-1206
- added JC2: SWTCHCRFT_3.5JACK5-JACK-SMD, jmsaavedra:SWTCHCRFT_3.5JACK5-JACK-SMD
- added L17: Grn, adafruit:LEDSMT1206
- added LED_: LED_RGB_PLCC-6, SpaceDIY_passive_components:LED_RGB_PLCC-6
- added PH34: (no value), pinhead:PINHD-1X1
- added PH64: (no value), pinhead:PINHD-1X3
- added PH65: (no value), pinhead:PINHD-1X4
- C21, C23, C24, C25, C26: device resistor:C-USC1206 -> SpaceDIY_passive_components:C0603
- C22: value 100n -> 470n
- PH21: device pinhead:PINHD-1X3 -> pinhead:PINHD-1X2
- PH31: device pinhead:PINHD-1X4 -> pinhead:PINHD-1X30
- PH38: device pinhead:PINHD-1X6 -> pinhead:PINHD-1X3
- R39: value 100k -> 330; device SpaceDIY_passive_components:R0603 -> resistor:R-US_R1206
- R40: value 1M -> 10k
- R60: device resistor:R-US_R1206 -> SpaceDIY_passive_components:R0603
- U2: value USB-B -> GAS_SENSOR; device SparkFun-Connectors:USBPTH -> SparkFun:GAS_SENSOR
Connections:
- removed net +OUT: IC11.+OUT_R, PH38.5
- removed net -OUT: IC11.-OUT_R, PH38.6
- removed net IN: C26.1, PH38.1
- removed net N$258: PH59.1, PH60.1, PH61.1
- removed net N$259: PH59.2, PH60.2, PH61.2
- removed net N$260: PH59.3, PH60.3, PH61.3
- removed net N$261: PH59.4, PH60.4, PH61.4
- removed net N$265: PH59.5, PH60.5, PH61.5
- removed net N$266: PH59.6, PH60.6, PH61.6
- removed net N$267: PH59.7, PH60.7, PH61.7
- removed net N$268: PH59.8, PH60.8, PH61.8
- removed net N$269: PH59.9, PH60.9, PH61.9
- removed net N$270: PH59.10, PH60.10, PH61.10
- removed net N$271: PH59.11, PH60.11, PH61.11
- removed net N$272: PH59.12, PH60.12, PH61.12
- removed net N$273: PH59.13, PH60.13, PH61.13
- removed net N$274: PH59.14, PH60.14, PH61.14
- removed net N$275: PH59.15, PH60.15, PH61.15
- removed net N$276: PH59.16, PH60.16, PH61.16
- removed net N$277: PH59.17, PH60.17, PH61.17
- removed net N$278: PH59.18, PH60.18, PH61.18
- removed net N$279: PH59.19, PH60.19, PH61.19
- removed net N$280: PH59.20, PH60.20, PH61.20
- removed net N$281: PH59.21, PH60.21, PH61.21
- removed net N$282: PH59.22, PH60.22, PH61.22
- removed net N$283: PH59.23, PH60.23, PH61.23
- removed net N$284: PH59.24, PH60.24, PH61.24
- removed net N$285: PH59.25, PH60.25, PH61.25
- removed net N$286: PH59.26, PH60.26, PH61.26
- removed net N$287: PH59.27, PH60.27, PH61.27
- removed net N$288: PH59.28, PH60.28, PH61.28
- removed net N$289: PH59.29, PH60.29, PH61.29
- removed net N$290: PH59.30, PH60.30, PH61.30
- removed net OUT01: IC9.OUT, PH21.2, R39.2
- removed net PVDD: C23.1, C24.1, C27.+, IC11.PVDD, IC11.PVDD1, IC11.VDD, PH38.3
- removed net SENSE: R67.1, U$15.0
- removed net SNS: C28.2, IC9.SNS, R40.2
- removed net SNSK: C28.1, IC9.SNSK, R67.2
- new net INL: IC11.INL, R60.1
- new net IN_L: C26.1, PH38.3
- new net IN_R: C22.1, PH38.2
- new net JC2: JC2.2, PH64.2
- new net N$118: F1.1, S1.LC
- new net N$119: PH34.1, R67.2, U2.B1
- new net N$120: JC2.1, PH64.3
- new net N$121: JC2.3, PH64.1
- new net N$122: L17.A, R39.1
- new net N$124: C22.2, R40.2
- new net N$127: PH31.7, PH59.7, PH60.7, PH61.7
- new net N$128: PH31.1, PH59.1, PH60.1, PH61.1
- new net N$129: PH31.2, PH59.2, PH60.2, PH61.2
- new net N$139: PH31.3, PH59.3, PH60.3, PH61.3
- new net N$140: PH31.4, PH59.4, PH60.4, PH61.4
- new net N$141: PH31.5, PH59.5, PH60.5, PH61.5
- new net N$142: PH31.6, PH59.6, PH60.6, PH61.6
- new net N$143: PH31.8, PH59.8, PH60.8, PH61.8
- new net N$144: PH31.9, PH59.9, PH60.9, PH61.9
- new net N$145: PH31.10, PH59.10, PH60.10, PH61.10
- new net N$147: PH31.11, PH59.11, PH60.11, PH61.11
- new net N$148: PH31.12, PH59.12, PH60.12, PH61.12
- new net N$149: PH31.13, PH59.13, PH60.13, PH61.13
- new net N$150: PH31.14, PH59.14, PH60.14, PH61.14
- new net N$151: PH31.15, PH59.15, PH60.15, PH61.15
- new net N$152: PH31.16, PH59.16, PH60.16, PH61.16
- new net N$153: PH31.17, PH59.17, PH60.17, PH61.17
- new net N$154: PH31.18, PH59.18, PH60.18, PH61.18
- new net N$163: PH31.19, PH59.19, PH60.19, PH61.19
- new net N$164: PH31.20, PH59.20, PH60.20, PH61.20
- new net N$165: PH31.21, PH59.21, PH60.21, PH61.21
- new net N$166: PH31.22, PH59.22, PH60.22, PH61.22
- new net N$167: PH31.23, PH59.23, PH60.23, PH61.23
- new net N$168: PH31.24, PH59.24, PH60.24, PH61.24
- new net N$169: PH31.25, PH59.25, PH60.25, PH61.25
- new net N$170: PH31.26, PH59.26, PH60.26, PH61.26
- new net N$174: PH31.27, PH59.27, PH60.27, PH61.27
- new net N$175: PH31.28, PH59.28, PH60.28, PH61.28
- new net N$176: PH31.29, PH59.29, PH60.29, PH61.29
- new net N$177: PH31.30, PH59.30, PH60.30, PH61.30
- new net OUT_L+: IC11.+OUT_L, PH65.4
- new net OUT_L-: IC11.-OUT_L, PH65.3
- new net OUT_R+: IC11.+OUT_R, PH65.2
- new net OUT_R-: IC11.-OUT_R, PH65.1
- net GND: now also L17.C, LED_B.C, LED_G.C, LED_R.C, PH38.1, R67.1, U2.H2; no longer C22.2, IC9.GND, IC9.TIME, PH38.2, PH38.4, R39.1, R40.1, RGBRGB-B.C, RGBRGB-G.C, RGBRGB-R.C, U2.GND
- net INR: now also R40.1; no longer R60.1
- net N$117: now also LED_G.A; no longer RGBRGB-G.A
- net N$126: now also PH21.2; no longer PH21.3
- net N$224: now also R39.2
- net N$308: now also LED_R.A; no longer RGBRGB-R.A
- net N$310: now also LED_B.A; no longer RGBRGB-B.A
- net SA': no longer PH31.1
- net SB': no longer PH13.1
- net SC': no longer PH13.3
- net SD': no longer PH31.4
- net SE': no longer PH31.3
- net SF': no longer PH31.2
- net SG': no longer PH13.2
- net VCC: now also C23.1, C24.1, C27.+, F1.2, IC11.PVDD, IC11.PVDD1, IC11.VDD, U2.A1, U2.H1; no longer C22.1, IC9.VDD, S1.LC
- net VUSB: no longer U2.VBUS
Other:
- note added: "Aux Interface"
- note added: "Sensor de gas"
- note added: "Sensor táctil"
- note removed: "CTI Robotics Interface"
- note removed: "Sensores táctiles"
- moved on the sheet: C23, C24, C25, C26, C27, L0, L1, L2, L3, L4, L5, L6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

Commit message: Updated to R3 (Mk.III)
Connections:
- net G: now also R57.2; no longer R58.2
- net R: now also R58.2; no longer R57.2
Changed lines of the file:
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@@
 </segment>
 <segment>
-<pinref part="R58" gate="G$1" pin="2"/>
-<wire x1="58.42" y1="22.86" x2="66.04" y2="22.86" width="0.1524" layer="91"/>
-<label x="58.42" y="22.86" size="1.778" layer="95"/>
+<pinref part="R57" gate="G$1" pin="2"/>
+<wire x1="58.42" y1="30.48" x2="66.04" y2="30.48" width="0.1524" layer="91"/>
+<label x="58.42" y="30.48" size="1.778" layer="95"/>
 </segment>
 </net>
@@
 </segment>
 <segment>
-<pinref part="R57" gate="G$1" pin="2"/>
-<wire x1="58.42" y1="30.48" x2="66.04" y2="30.48" width="0.1524" layer="91"/>
-<label x="58.42" y="30.48" size="1.778" layer="95"/>
+<pinref part="R58" gate="G$1" pin="2"/>
+<wire x1="58.42" y1="22.86" x2="66.04" y2="22.86" width="0.1524" layer="91"/>
+<label x="58.42" y="22.86" size="1.778" layer="95"/>
 </segment>
 </net>
